Commit message: feat: Add laser scan

File: description/edubot_core.xacro (robot description, xacro)
@@ -17,4 +17,7 @@
         <color rgba="0 0 0 1" />
     </material>
+    <material name="red">
+        <color rgba="1 0 0 1" />
+    </material>
     <!-- BASE LINK  -->
     <link name="base_link">

File: description/robot.urdf.xacro (robot description, xacro)
@@ -4,3 +4,4 @@
     <xacro:include filename="edubot_core.xacro" />
     <xacro:include filename="gazebo_control.xacro" />
+    <xacro:include filename="lidar.xacro" />
 </robot>
